Commit message: Update test_bot.xacro

File: tortoisebot_description/urdf/test_bot.xacro (robot description, xacro)
@@ -10,5 +10,5 @@
 	</joint>
 	<joint name="lidar_joint" type="fixed">
-		<origin rpy="0 0 0" xyz="-0.02 0.0 0.4"/>
+		<origin rpy="0 0 0" xyz="-0.2 0.0 0.4"/>
 		<parent link="base_link"/>
 		<child link="lidar"/>
