Commit message: Update for gazebo sim ignition ( fortress)

File: tortoisebot_description/models/urdf/tortoisebot_simple.xacro (robot description, xacro)
@@ -122,16 +122,16 @@
     <origin xyz="2.5326962749261384e-14 4.504651888394023e-14 -0.0017582044401419582" rpy="0 0 0"/>
     <mass value="0.0033567272126794434"/>
-    <inertia ixx="0.0" iyy="0.0" izz="0.0" ixy="0.0" iyz="0.0" ixz="0.0"/>
+    <inertia ixx="1e-06" iyy="1e-06" izz="1e-06" ixy="0.0" iyz="0.0" ixz="0.0"/>
   </inertial>
   <visual>
-    <origin xyz="0.0767 0.0 -0.0049" rpy="0 0 0"/>
+    <origin xyz="-0.0000 0.0 0.0005" rpy="0 0 0"/>
     <geometry>
-      <mesh filename="file://$(find tortoisebot_description)/models/meshes/castor_wheel.dae" scale="0.001 0.001 0.001"/>
+      <sphere radius="0.005"/>
     </geometry>
   </visual>
   <collision>
-    <origin xyz="0.0767 0.0 -0.0049" rpy="0 0 0"/>
+    <origin xyz="-0.0000 0.0 0.0005" rpy="0 0 0"/>
     <geometry>
-      <mesh filename="file://$(find tortoisebot_description)/models/meshes/castor_wheel.dae" scale="0.001 0.001 0.001"/>
+      <sphere radius="0.005"/>
     </geometry>
   </collision>

Commit message: update for ros2 jazzy with gazebo garden support in sim

File: tortoisebot_description/models/urdf/tortoisebot_simple.xacro (robot description, xacro)
@@ -19,5 +19,5 @@
     <origin xyz="0 0 0" rpy="0 0 0"/>
     <geometry>
-      <mesh filename="file://$(find tortoisebot_description)/models/meshes/base_link.dae" scale="0.001 0.001 0.001"/>
+      <mesh filename="file://$(find tortoisebot_description)/models/meshes/convex_base_link.dae" scale="0.001 0.001 0.001"/>
     </geometry>
   </collision>
@@ -38,5 +38,5 @@
     <origin xyz="0.000197 -0.0778 -0.032453" rpy="0 0 0"/>
     <geometry>
-      <mesh filename="file://$(find tortoisebot_description)/models/meshes/wheel_left.dae" scale="0.001 0.001 0.001"/>
+      <mesh filename="file://$(find tortoisebot_description)/models/meshes/convex_wheel_left.dae" scale="0.001 0.001 0.001"/>
     </geometry>
   </collision>
@@ -57,5 +57,5 @@
     <origin xyz="-0.0001 0.0778 -0.032453" rpy="0 0 0"/>
     <geometry>
-      <mesh filename="file://$(find tortoisebot_description)/models/meshes/wheel_right.dae" scale="0.001 0.001 0.001"/>
+      <mesh filename="file://$(find tortoisebot_description)/models/meshes/convex_wheel_right.dae" scale="0.001 0.001 0.001"/>
     </geometry>
   </collision>
@@ -76,5 +76,5 @@
     <origin xyz="0.03275 0.0 -0.167" rpy="0 0 0"/>
     <geometry>
-      <mesh filename="file://$(find tortoisebot_description)/models/meshes/lidar.dae" scale="0.001 0.001 0.001"/>
+      <mesh filename="file://$(find tortoisebot_description)/models/meshes/convex_lidar.dae" scale="0.001 0.001 0.001"/>
     </geometry>
   </collision>
@@ -95,5 +95,5 @@
     <origin xyz="-0.05025 -1e-05 -0.133907" rpy="0 0 0"/>
     <geometry>
-      <mesh filename="file://$(find tortoisebot_description)/models/meshes/camera_link.dae" scale="0.001 0.001 0.001"/>
+      <mesh filename="file://$(find tortoisebot_description)/models/meshes/convex_camera_link.dae" scale="0.001 0.001 0.001"/>
     </geometry>
   </collision>
@@ -114,5 +114,5 @@
     <origin xyz="-0.03125 0.0 -0.131063" rpy="0 0 0"/>
     <geometry>
-      <mesh filename="file://$(find tortoisebot_description)/models/meshes/camera_holder.dae" scale="0.001 0.001 0.001"/>
+      <mesh filename="file://$(find tortoisebot_description)/models/meshes/convex_camera_holder.dae" scale="0.001 0.001 0.001"/>
     </geometry>
   </collision>
@@ -122,16 +122,16 @@
     <origin xyz="2.5326962749261384e-14 4.504651888394023e-14 -0.0017582044401419582" rpy="0 0 0"/>
     <mass value="0.0033567272126794434"/>
-    <inertia ixx="0.0" iyy="0.0" izz="0.0" ixy="0.0" iyz="0.0" ixz="0.0"/>
+    <inertia ixx="1e-06" iyy="1e-06" izz="1e-06" ixy="0.0" iyz="0.0" ixz="0.0"/>
   </inertial>
   <visual>
-    <origin xyz="0.0767 0.0 -0.0049" rpy="0 0 0"/>
+    <origin xyz="-0.0000 0.0 0.0005" rpy="0 0 0"/>
     <geometry>
-      <mesh filename="file://$(find tortoisebot_description)/models/meshes/castor_wheel.dae" scale="0.001 0.001 0.001"/>
+      <sphere radius="0.005"/>
     </geometry>
   </visual>
   <collision>
-    <origin xyz="0.0767 0.0 -0.0049" rpy="0 0 0"/>
+    <origin xyz="-0.0000 0.0 0.0005" rpy="0 0 0"/>
     <geometry>
-      <mesh filename="file://$(find tortoisebot_description)/models/meshes/castor_wheel.dae" scale="0.001 0.001 0.001"/>
+      <sphere radius="0.005"/>
     </geometry>
   </collision>
